Commit message: Changes to xacro file to add the depth camera link, removed tutorial_pkg

File: src/rosbot_description/urdf/rosbot.xacro (robot description, xacro)
@@ -283,4 +283,10 @@
   <link name="camera_depth_frame">
   </link>
+  <joint name="camera_depth_optical_joint" type="fixed">
+    <origin xyz="0 0 0" rpy="-1.5708 0 -1.5708" />
+    <parent link="camera_depth_frame" />
+    <child link="camera_depth_optical_frame" />
+  </joint>
+  <link name="camera_depth_optical_frame"/>
   <joint name="rplidar_joint" type="fixed">
     <axis xyz="0 1 0" />

Commit message: Rosbot urdf changed per new design

File: src/rosbot_description/urdf/rosbot.xacro (robot description, xacro)
@@ -246,5 +246,5 @@
   <joint name="astra_joint" type="fixed">
     <axis xyz="0 0 0" />
-    <origin xyz="-0.03 0 0.18" rpy="0 0 0"/>
+    <origin xyz="0.11 0 0.096" rpy="0 0 0"/>
     <parent link="base_link"/>
     <child link="camera_link"/>
@@ -260,5 +260,5 @@
       <origin xyz="-0.01 0 -0.03" rpy="1.5707 0 1.5707"/>
       <geometry>
-        <mesh filename="package://rosbot_description/meshes/astra.dae" scale="0.001 0.001 0.001" />
+        <mesh filename="package://rosbot_description/meshes/astra_minimal.dae" scale="0.001 0.001 0.001" />
       </geometry>
     </visual>
@@ -291,5 +291,5 @@
   <joint name="rplidar_joint" type="fixed">
     <axis xyz="0 1 0" />
-    <origin xyz="0.02 0 0" rpy="0 0 3.14"/>
+    <origin xyz="0.02 0 0.0157" rpy="0 0 3.14"/>
     <parent link="base_link"/>
     <child link="laser"/>

Commit message: Added tracker in urdf, colors changed

File: src/rosbot_description/urdf/rosbot.xacro (robot description, xacro)
@@ -343,3 +343,24 @@
   </joint>
   <link name="range_rr"></link>
+  <!-- HTC Vive, only for visuals-->
+  <joint name="vive_joint" type="fixed">
+    <axis xyz="0 0 0" />
+    <origin xyz="-0.03 0 0.14" rpy="0 0 0"/>
+    <parent link="base_link"/>
+    <child link="vive"/>
+  </joint>
+  <link name="vive">
+    <collision>
+      <origin xyz="0 0 0" rpy="0 0 0"/>
+      <geometry>
+        <mesh filename="package://rosbot_description/meshes/htc_vive_tracker.dae" scale="0.001 0.001 0.001" />
+      </geometry>
+    </collision>
+    <visual>
+      <origin xyz="0 0 0" rpy="0 0 0"/>
+      <geometry>
+        <mesh filename="package://rosbot_description/meshes/htc_vive_tracker.dae" scale="0.001 0.001 0.001" />
+      </geometry>
+    </visual>
+  </link>
 </robot>

Commit message: fixed somw urdf issue for gazebo11

File: src/rosbot_description/urdf/rosbot.xacro (robot description, xacro)
@@ -7,4 +7,10 @@
   <xacro:include filename="$(find rosbot_description)/urdf/materials.xacro" />
   <xacro:include filename="$(find rosbot_description)/urdf/macros.xacro" />
+  <link name="dummy">
+   </link>
+  <joint name="dummy_joint" type="fixed">
+     <parent link="dummy"/>
+     <child link="base_link"/>
+   </joint>
   <link name='base_link'>
     <pose>0 0 0.1 0 0 0</pose>
